File: ESP32-Antennenschalter.kicad_sch (KiCad schematic)
At the start: 117 parts, among them J1 IN1(TRX1), J10 T1_In, J11 T1_Out, J12 T2_Out, J13 T2_In, J14 Tuner/Ext_TRX, J15 Tuner/Ext_ANT, J16 L2, J17 L2, J18 L2, J19 L2, J2 IN2(TRX2), J20 L2, J21 L2, J22 L2, J23 L2, J24 MCP_Addr, J25 ADC2, J26 ADC3, J27 Ext, J28 ADC_Addr, J3 IN3(RX), J4 ANT1, J5 ANT2, J6 ANT3, J7 ANT4, J8 ANT-DUMMY, J9 ANT-RX, K1 Finder 40.31.6.006.0000, K10 Finder 40.31.6.006.0000, K11 Finder 40.31.6.006.0000, K12 Finder 40.31.6.006.0000, K13 Finder 40.31.6.006.0000, K14 Finder 40.31.6.006.0000, K15 Finder 40.31.6.006.0000, K16 Finder 40.31.6.006.0000, K2 Finder 40.31.6.006.0000, K3 Finder 40.31.6.006.0000, K4 Finder 40.31.6.006.0000, K5 Finder 40.31.6.006.0000, K6 Finder 40.31.6.006.0000, K7 Finder 40.31.6.006.0000, K8 Finder 40.31.6.006.0000, K9 Finder 40.31.6.006.0000, SW1 Input, SW2 Output, U2 DRV8833PWP, U3 DRV8833PWP, U4 MCP23017_SO, U5 DRV8833PWP, U6 DRV8833PWP, U7 ADS1115IDGS, U8 Wemos D1 mini ESP32

Commit message: Add files via upload
Parts:
- added J29, J30, J31, J32, J33, J34, J35, J36, J37, J38, J39, J40, J41, J42, J43, J44: Conn_01x01_Pin, Connector_Pin:Pin_D0.7mm_L6.5mm_W1.8mm_FlatFork, symbol Connector:Conn_01x01_Pin
Connections:
- net GND: now also J29.1 (Pin_1), J30.1 (Pin_1), J31.1 (Pin_1), J32.1 (Pin_1), J33.1 (Pin_1), J34.1 (Pin_1), J35.1 (Pin_1), J36.1 (Pin_1), J37.1 (Pin_1), J38.1 (Pin_1), J39.1 (Pin_1), J40.1 (Pin_1), J41.1 (Pin_1), J42.1 (Pin_1), J43.1 (Pin_1), J44.1 (Pin_1)
Other:
- moved on the sheet: H1, H2, H3, H4, H5

Commit message: SWR-Meter: Remove R11,R23; Replace R4,R5 with 8.2K
Parts:
- R11, R12: value 100k -> REMOVE
- R4, R5: value 100k -> 8.2k
Other:
- note added: "(max 10.6V)"
- note added: "(max 220W)"
- note removed: "(max 200W)"
Changed lines of the file:
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@@
 		)
 	)
+	(text "(max 10.6V)"
+		(exclude_from_sim no)
+		(at 139.446 58.42 90)
+		(effects
+			(font
+				(size 1.27 1.27)
+				(thickness 0.254)
+				(bold yes)
+			)
+		)
+	)
 	(text "0x20"
 		(exclude_from_sim no)
@@
 		)
 	)
-	(text "(max 200W)"
+	(text "(max 220W)"
 		(exclude_from_sim no)
 		(at 138.684 26.162 90)
@@
 			)
 		)
-		(property "Value" "100k"
+		(property "Value" "8.2k"
 			(at 147.32 73.66 0)
 			(effects
@@
 			)
 		)
-		(property "Value" "100k"
+		(property "Value" "REMOVE"
 			(at 147.574 88.646 90)
 			(effects
@@
 			)
 		)
-		(property "Value" "100k"
+		(property "Value" "8.2k"
 			(at 162.56 73.914 0)
 			(effects
@@
 			)
 		)
-		(property "Value" "100k"
+		(property "Value" "REMOVE"
 			(at 162.814 88.646 90)
 			(effects
